File: board1.kicad_pcb (KiCad board)
At the start: 0 parts

Commit message: Created Physical Board Layout
Created Edge Cuts for Physical Board
Layout based off of Rushil's drawing
Other:
- board outline added: 99.3 x 99.3 mm
- copper layers 0 -> 2
- board text added: "circles are arbitrary radius, can be resized for mounting holes later do not edit for now, if need be, just change radius"
Changed lines of the file:
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@@
 (kicad_pcb (version 20211014) (generator pcbnew)
+  (general
+    (thickness 1.6)
+  )
+  (paper "A4")
+  (layers
+    (0 "F.Cu" signal)
+    (31 "B.Cu" signal)
+    (32 "B.Adhes" user "B.Adhesive")
+    (33 "F.Adhes" user "F.Adhesive")
+    (34 "B.Paste" user)
+    (35 "F.Paste" user)
+    (36 "B.SilkS" user "B.Silkscreen")
+    (37 "F.SilkS" user "F.Silkscreen")
+    (38 "B.Mask" user)
+    (39 "F.Mask" user)
+    (40 "Dwgs.User" user "User.Drawings")
+    (41 "Cmts.User" user "User.Comments")
+    (42 "Eco1.User" user "User.Eco1")
+    (43 "Eco2.User" user "User.Eco2")
+    (44 "Edge.Cuts" user)
+    (45 "Margin" user)
+    (46 "B.CrtYd" user "B.Courtyard")
+    (47 "F.CrtYd" user "F.Courtyard")
+    (48 "B.Fab" user)
+    (49 "F.Fab" user)
+    (50 "User.1" user)
+    (51 "User.2" user)
+    (52 "User.3" user)
+    (53 "User.4" user)
+    (54 "User.5" user)
+    (55 "User.6" user)
+    (56 "User.7" user)
+    (57 "User.8" user)
+    (58 "User.9" user)
+  )
+  (setup
+    (pad_to_mask_clearance 0)
+    (pcbplotparams
+      (layerselection 0x00010fc_ffffffff)
+      (disableapertmacros false)
+      (usegerberextensions false)
+      (usegerberattributes true)
+      (usegerberadvancedattributes true)
+      (creategerberjobfile true)
+      (svguseinch false)
+      (svgprecision 6)
+      (excludeedgelayer true)
+      (plotframeref false)
+      (viasonmask false)
+      (mode 1)
+      (useauxorigin false)
+      (hpglpennumber 1)
+      (hpglpenspeed 20)
+      (hpglpendiameter 15.000000)
+      (dxfpolygonmode true)
+      (dxfimperialunits true)
+      (dxfusepcbnewfont true)
+      (psnegative false)
+      (psa4output false)
+      (plotreference true)
+      (plotvalue true)
+      (plotinvisibletext false)
+      (sketchpadsonfab false)
+      (subtractmaskfromsilk false)
+      (outputformat 1)
+      (mirror false)
+      (drillshape 1)
+      (scaleselection 1)
+      (outputdirectory "")
+    )
+  )
+  (net 0 "")
+  (gr_line (start 91.5924 70.0076) (end 91.5924 149.2556) (layer "Edge.Cuts") (width 0.1))
+  (gr_circle (center 101.6 70.0076) (end 110.49 70.0076) (layer "Edge.Cuts") (width 0.1) (fill none))
+  (gr_line (start 190.8556 70.0076) (end 190.8556 149.2556) (layer "Edge.Cuts") (width 0.1))
+  (gr_circle (center 101.6 149.2556) (end 110.49 149.2556) (layer "Edge.Cuts") (width 0.1) (fill none))
+  (gr_line (start 101.6 159.2632) (end 180.848 159.2632) (layer "Edge.Cuts") (width 0.1))
+  (gr_line (start 101.6 60) (end 180.848 60) (layer "Edge.Cuts") (width 0.1))
+  (gr_circle (center 180.848 149.2556) (end 189.738 149.2556) (layer "Edge.Cuts") (width 0.1) (fill none))
+  (gr_circle (center 180.848 70.0076) (end 189.738 70.0076) (layer "Edge.Cuts") (width 0.1) (fill none))
+  (gr_arc (start 190.8556 149.2556) (mid 187.924442 156.332042) (end 180.848 159.2632) (layer "Edge.Cuts") (width 0.1))
+  (gr_arc (start 101.6 159.2632) (mid 94.523558 156.332042) (end 91.5924 149.2556) (layer "Edge.Cuts") (width 0.1))
+  (gr_arc (start 180.848 60) (mid 187.924442 62.931158) (end 190.8556 70.0076) (layer "Edge.Cuts") (width 0.1))
+  (gr_arc (start 91.5924 70.0076) (mid 94.523558 62.931158) (end 101.6 60) (layer "Edge.Cuts") (width 0.1))
+  (gr_text "circles are arbitrary radius, can be resized for mounting holes later\ndo not edit for now, if need be, just change radius\n" (at 139 54) (layer "Edge.Cuts")
+    (effects (font (size 1 1) (thickness 0.15)))
+  )
 )
