File: board1.kicad_pcb (KiCad board)
At the start: 4 copper layers, 101.2 x 101.2 mm, 24 parts, among them J6 XT30 Male Connector, U1 BNO085, U2 Teensy_4.0, U3 Raspberry_PI_Zero_W, U4 D24V50F5

Commit message: additional changes
Other:
- board text removed: "circles are arbitrary radius, can be resized for mounting holes later do not edit for now, if need be, just change radius"
Changed lines of the file:
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@@
   (gr_arc (start 96.0434 63.8356) (mid 99.264698 56.058698) (end 107.0416 52.8374) (layer "Edge.Cuts") (width 0.1))
   (gr_circle (center 186.2896 63.8356) (end 188.982 63.8356) (layer "Edge.Cuts") (width 0.1) (fill none))
-  (gr_text "circles are arbitrary radius, can be resized for mounting holes later\ndo not edit for now, if need be, just change radius\n" (at 144.4416 46.8374) (layer "Edge.Cuts")
-    (effects (font (size 1 1) (thickness 0.15)))
-  )
   (segment (start 136.65 109.25) (end 131.9 109.25) (width 0.5) (layer "B.Cu") (net 1))
   (segment (start 131.05 108.4) (end 131.05 104.4) (width 0.5) (layer "B.Cu") (net 1))
@@
   (zone (net 20) (net_name "/12V") (layer "In2.Cu") (hatch edge 0.508)
     (connect_pads (clearance 0.508))
-    (min_thickness 0.254)
-    (fill (thermal_gap 0.508) (thermal_bridge_width 0.508))
+    (min_thickness 0.254) (filled_areas_thickness no)
+    (fill yes (thermal_gap 0.508) (thermal_bridge_width 0.508))
     (polygon
       (pts
