File: board1.kicad_sch (KiCad schematic)
At the start: 24 parts, among them J6 XT30 Male Connector, U1 BNO085, U2 Teensy_4.0, U3 Raspberry_PI_Zero_W, U4 D24V50F5

Commit message: preliminary routing of traces
Connections:
- net 5V: now also U3.4 (5V)
- net BATTERY_GROUND: now also U4.3 (GND)
- net GNDREF: now also U2.4 (GND), U3.14 (GND), U3.20 (GND), U3.25 (GND), U3.30 (GND), U3.34 (GND), U3.39 (GND), U3.9 (GND)
- no-connect marks 63 -> 57
Changed lines of the file:
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@@
   (no_connect (at 184.15 50.8))
   (no_connect (at 184.15 53.34))
+  (no_connect (at 227.33 93.98))
   (no_connect (at 293.37 38.1))
   (no_connect (at 316.23 53.34))
   (no_connect (at 316.23 50.8))
   (no_connect (at 293.37 53.34))
-  (no_connect (at 332.74 139.7))
-  (no_connect (at 184.15 78.74))
+  (no_connect (at 184.15 86.36))
+  (no_connect (at 184.15 83.82))
+  (no_connect (at 227.33 91.44))
   (no_connect (at 332.74 144.78))
   (no_connect (at 316.23 83.82))
@@
   (no_connect (at 64.77 125.73))
   (no_connect (at 375.92 81.28))
-  (no_connect (at 99.06 45.72))
   (no_connect (at 377.19 53.34))
   (no_connect (at 375.92 78.74))
@@
   (no_connect (at 293.37 68.58))
   (no_connect (at 227.33 96.52))
-  (no_connect (at 227.33 88.9))
   (no_connect (at 184.15 48.26))
   (no_connect (at 184.15 88.9))
-  (no_connect (at 184.15 96.52))
   (no_connect (at 184.15 91.44))
   (no_connect (at 184.15 93.98))
-  (no_connect (at 184.15 58.42))
   (no_connect (at 184.15 60.96))
   (no_connect (at 184.15 55.88))
@@
   (no_connect (at 227.33 66.04))
   (no_connect (at 227.33 60.96))
-  (no_connect (at 227.33 63.5))
-  (no_connect (at 227.33 83.82))
   (no_connect (at 227.33 81.28))
   (no_connect (at 227.33 78.74))
@@
   (no_connect (at 227.33 86.36))
   (no_connect (at 227.33 73.66))
-  (no_connect (at 227.33 71.12))
-  (no_connect (at 227.33 50.8))
   (no_connect (at 353.06 68.58))
   (no_connect (at 293.37 83.82))
@@
     (effects (font (size 1.27 1.27)) (justify left bottom))
   )
+  (label "5V" (at 227.33 50.8 0)
+    (effects (font (size 1.27 1.27)) (justify left bottom))
+  )
   (label "BATTERY_GROUND" (at 316.23 40.64 0)
     (effects (font (size 1.27 1.27)) (justify left bottom))
@@
     (effects (font (size 1.27 1.27)) (justify right bottom))
   )
+  (label "BATTERY_GROUND" (at 332.74 139.7 180)
+    (effects (font (size 1.27 1.27)) (justify right bottom))
+  )
   (label "ENC_2_PINB" (at 50.8 53.34 180)
     (effects (font (size 1.27 1.27)) (justify right bottom))
@@
   (label "ENC_3_PINA" (at 302.26 232.41 0)
     (effects (font (size 1.27 1.27)) (justify left bottom))
+  )
+  (symbol (lib_id "power:GNDREF") (at 184.15 96.52 270) (unit 1)
+    (in_bom yes) (on_board yes) (fields_autoplaced)
+    (property "Reference" "#PWR0118" (id 0) (at 177.8 96.52 0)
+      (effects (font (size 1.27 1.27)) hide)
+    )
+    (property "Value" "GNDREF" (id 1) (at 180.34 96.5199 90)
+      (effects (font (size 1.27 1.27)) (justify right))
+    )
+    (property "Footprint" "" (id 2) (at 184.15 96.52 0)
+      (effects (font (size 1.27 1.27)) hide)
+    )
+    (property "Datasheet" "" (id 3) (at 184.15 96.52 0)
+      (effects (font (size 1.27 1.27)) hide)
+    )
+    (pin "1")
   )
   (symbol (lib_id "Connector:Conn_01x02_Female") (at 58.42 229.87 180) (unit 1)
@@
     (pin "1")
   )
+  (symbol (lib_id "power:GNDREF") (at 227.33 83.82 90) (unit 1)
+    (in_bom yes) (on_board yes) (fields_autoplaced)
+    (property "Reference" "#PWR0116" (id 0) (at 233.68 83.82 0)
+      (effects (font (size 1.27 1.27)) hide)
+    )
+    (property "Value" "GNDREF" (id 1) (at 231.14 83.8199 90)
+      (effects (font (size 1.27 1.27)) (justify right))
+    )
+    (property "Footprint" "" (id 2) (at 227.33 83.82 0)
+      (effects (font (size 1.27 1.27)) hide)
+    )
+    (property "Datasheet" "" (id 3) (at 227.33 83.82 0)
+      (effects (font (size 1.27 1.27)) hide)
+    )
+    (pin "1")
+  )
   (symbol (lib_id "Connector:Conn_01x06_Male") (at 297.18 229.87 0) (unit 1)
     (in_bom yes) (on_board yes) (fields_autoplaced)
@@
     (pin "6")
   )
+  (symbol (lib_id "power:GNDREF") (at 184.15 78.74 270) (unit 1)
+    (in_bom yes) (on_board yes) (fields_autoplaced)
+    (property "Reference" "#PWR0119" (id 0) (at 177.8 78.74 0)
+      (effects (font (size 1.27 1.27)) hide)
+    )
+    (property "Value" "GNDREF" (id 1) (at 180.34 78.7399 90)
+      (effects (font (size 1.27 1.27)) (justify right))
+    )
+    (property "Footprint" "" (id 2) (at 184.15 78.74 0)
+      (effects (font (size 1.27 1.27)) hide)
+    )
+    (property "Datasheet" "" (id 3) (at 184.15 78.74 0)
+      (effects (font (size 1.27 1.27)) hide)
+    )
+    (pin "1")
+  )
   (symbol (lib_id "power:GNDREF") (at 82.55 133.35 90) (unit 1)
     (in_bom yes) (on_board yes) (fields_autoplaced)
@@
     (pin "1")
   )
+  (symbol (lib_id "power:GNDREF") (at 227.33 63.5 90) (unit 1)
+    (in_bom yes) (on_board yes) (fields_autoplaced)
+    (property "Reference" "#PWR0112" (id 0) (at 233.68 63.5 0)
+      (effects (font (size 1.27 1.27)) hide)
+    )
+    (property "Value" "GNDREF" (id 1) (at 231.14 63.4999 90)
+      (effects (font (size 1.27 1.27)) (justify right))
+    )
+    (property "Footprint" "" (id 2) (at 227.33 63.5 0)
+      (effects (font (size 1.27 1.27)) hide)
+    )
+    (property "Datasheet" "" (id 3) (at 227.33 63.5 0)
+      (effects (font (size 1.27 1.27)) hide)
+    )
+    (pin "1")
+  )
   (symbol (lib_id "power:GNDREF") (at 293.37 48.26 270) (unit 1)
     (in_bom yes) (on_board yes) (fields_autoplaced)
@@
     )
     (property "Datasheet" "" (id 3) (at 239.395 53.34 0)
+      (effects (font (size 1.27 1.27)) hide)
+    )
+    (pin "1")
+  )
+  (symbol (lib_id "power:GNDREF") (at 227.33 71.12 90) (unit 1)
+    (in_bom yes) (on_board yes) (fields_autoplaced)
+    (property "Reference" "#PWR0115" (id 0) (at 233.68 71.12 0)
+      (effects (font (size 1.27 1.27)) hide)
+    )
+    (property "Value" "GNDREF" (id 1) (at 231.14 71.1199 90)
+      (effects (font (size 1.27 1.27)) (justify right))
+    )
+    (property "Footprint" "" (id 2) (at 227.33 71.12 0)
+      (effects (font (size 1.27 1.27)) hide)
+    )
+    (property "Datasheet" "" (id 3) (at 227.33 71.12 0)
       (effects (font (size 1.27 1.27)) hide)
     )
@@
     (pin "6")
   )
+  (symbol (lib_id "power:GNDREF") (at 184.15 58.42 270) (unit 1)
+    (in_bom yes) (on_board yes) (fields_autoplaced)
+    (property "Reference" "#PWR0114" (id 0) (at 177.8 58.42 0)
+      (effects (font (size 1.27 1.27)) hide)
+    )
+    (property "Value" "GNDREF" (id 1) (at 180.34 58.4199 90)
+      (effects (font (size 1.27 1.27)) (justify right))
+    )
+    (property "Footprint" "" (id 2) (at 184.15 58.42 0)
+      (effects (font (size 1.27 1.27)) hide)
+    )
+    (property "Datasheet" "" (id 3) (at 184.15 58.42 0)
+      (effects (font (size 1.27 1.27)) hide)
+    )
+    (pin "1")
+  )
   (symbol (lib_id "power:GNDREF") (at 354.33 40.64 270) (unit 1)
     (in_bom yes) (on_board yes)
@@
     (pin "1")
   )
+  (symbol (lib_id "power:GNDREF") (at 99.06 45.72 90) (unit 1)
+    (in_bom yes) (on_board yes) (fields_autoplaced)
+    (property "Reference" "#PWR0113" (id 0) (at 105.41 45.72 0)
+      (effects (font (size 1.27 1.27)) hide)
+    )
+    (property "Value" "GNDREF" (id 1) (at 102.87 45.7199 90)
+      (effects (font (size 1.27 1.27)) (justify right))
+    )
+    (property "Footprint" "" (id 2) (at 99.06 45.72 0)
+      (effects (font (size 1.27 1.27)) hide)
+    )
+    (property "Datasheet" "" (id 3) (at 99.06 45.72 0)
+      (effects (font (size 1.27 1.27)) hide)
+    )
+    (pin "1")
+  )
   (symbol (lib_id "power:GNDREF") (at 332.74 207.01 90) (unit 1)
     (in_bom yes) (on_board yes) (fields_autoplaced)
@@
     (pin "1")
   )
+  (symbol (lib_id "power:GNDREF") (at 227.33 88.9 90) (unit 1)
+    (in_bom yes) (on_board yes) (fields_autoplaced)
+    (property "Reference" "#PWR0117" (id 0) (at 233.68 88.9 0)
+      (effects (font (size 1.27 1.27)) hide)
+    )
+    (property "Value" "GNDREF" (id 1) (at 231.14 88.8999 90)
+      (effects (font (size 1.27 1.27)) (justify right))
+    )
+    (property "Footprint" "" (id 2) (at 227.33 88.9 0)
+      (effects (font (size 1.27 1.27)) hide)
+    )
+    (property "Datasheet" "" (id 3) (at 227.33 88.9 0)
+      (effects (font (size 1.27 1.27)) hide)
+    )
+    (pin "1")
+  )
   (symbol (lib_id "board1_libs:BNO085") (at 73.66 123.19 0) (unit 1)
     (in_bom yes) (on_board yes) (fields_autoplaced)
@@
     )
     (pin "")
-    (pin "4")
-    (pin "3")
-    (pin "12")
     (pin "")
     (pin "")
     (pin "")
+    (pin "1")
+    (pin "12")
+    (pin "2")
+    (pin "3")
+    (pin "4")
     (pin "5")
     (pin "6")
-    (pin "2")
     (pin "8")
-    (pin "1")
   )
   (symbol (lib_id "power:GNDREF") (at 55.88 250.19 90) (unit 1)
@@
       (reference "#PWR0111") (unit 1) (value "GNDREF") (footprint "")
     )
+    (path "/608b2c65-eb72-4945-8955-a01f5ffdbc0e"
+      (reference "#PWR0112") (unit 1) (value "GNDREF") (footprint "")
+    )
+    (path "/c54a43f7-4855-4b3b-8abb-2288a5920759"
+      (reference "#PWR0113") (unit 1) (value "GNDREF") (footprint "")
+    )
+    (path "/b9539c24-fe3d-4b51-abdf-150dec05fdc3"
+      (reference "#PWR0114") (unit 1) (value "GNDREF") (footprint "")
+    )
+    (path "/78552f95-7eea-4de3-a5c1-444f271c7bf4"
+      (reference "#PWR0115") (unit 1) (value "GNDREF") (footprint "")
+    )
+    (path "/0e7bb784-6e00-4b0f-9182-c08c4e02b1f4"
+      (reference "#PWR0116") (unit 1) (value "GNDREF") (footprint "")
+    )
+    (path "/dd81d22f-81c8-4eab-8e7e-c4ffab94b68d"
+      (reference "#PWR0117") (unit 1) (value "GNDREF") (footprint "")
+    )
+    (path "/042a8dc8-d4b7-4330-8371-b1c808008ef5"
+      (reference "#PWR0118") (unit 1) (value "GNDREF") (footprint "")
+    )
+    (path "/4a849690-dab5-4c38-a1c3-01574d61687c"
+      (reference "#PWR0119") (unit 1) (value "GNDREF") (footprint "")
+    )
     (path "/8885b28d-2bf8-468a-882c-f4b9524ec639"

Commit message: Updated PCB
Flipped Encoder, Increased Trace Size, and Changed Resistors to be 0805
Parts:
- R1, R2, R3: footprint board1_footprints:Resistor -> Resistor_SMD:R_0805_2012Metric
Changed lines of the file:
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@@
     (property "Reference" "R1" (id 0) (at 135.89 162.56 90))
     (property "Value" "4.7k" (id 1) (at 135.89 165.1 90))
-    (property "Footprint" "board1_footprints:Resistor" (id 2) (at 136.144 167.894 90)
+    (property "Footprint" "Resistor_SMD:R_0805_2012Metric" (id 2) (at 136.144 167.894 90)
       (effects (font (size 1.27 1.27)) hide)
     )
@@
     (property "Reference" "R3" (id 0) (at 200.66 132.08 90))
     (property "Value" "0 Ohms" (id 1) (at 200.66 134.62 90))
-    (property "Footprint" "board1_footprints:Resistor" (id 2) (at 200.914 137.414 90)
+    (property "Footprint" "Resistor_SMD:R_0805_2012Metric" (id 2) (at 200.914 137.414 90)
       (effects (font (size 1.27 1.27)) hide)
     )
@@
     (property "Reference" "R2" (id 0) (at 135.89 171.45 90))
     (property "Value" "4.7k" (id 1) (at 135.89 173.99 90))
-    (property "Footprint" "board1_footprints:Resistor" (id 2) (at 136.144 176.784 90)
+    (property "Footprint" "Resistor_SMD:R_0805_2012Metric" (id 2) (at 136.144 176.784 90)
       (effects (font (size 1.27 1.27)) hide)
     )
@@
     )
     (path "/cc5b2ee6-d349-4c1c-9750-94bfdf9bcb6a"
-      (reference "R1") (unit 1) (value "4.7k") (footprint "board1_footprints:Resistor")
+      (reference "R1") (unit 1) (value "4.7k") (footprint "Resistor_SMD:R_0805_2012Metric")
     )
     (path "/e57e32b3-419e-40f1-b3a9-e60718f08f65"
-      (reference "R2") (unit 1) (value "4.7k") (footprint "board1_footprints:Resistor")
+      (reference "R2") (unit 1) (value "4.7k") (footprint "Resistor_SMD:R_0805_2012Metric")
     )
     (path "/d2ff947e-532f-4c8e-b9db-65ba031f8106"
-      (reference "R3") (unit 1) (value "0 Ohms") (footprint "board1_footprints:Resistor")
+      (reference "R3") (unit 1) (value "0 Ohms") (footprint "Resistor_SMD:R_0805_2012Metric")
     )
     (path "/2d72a194-045f-4119-bc37-1519af19084d"
